File: Hardware/0. Project/WorkshySwitch.brd (EAGLE design)
At the start: 35 x 45 mm, 52 parts, among them K1 G3MB-202P, Q3 32-MHz, Q4 32.768-kHz, T1 BC848, U1 LM1117-3.3, U2 HLK-PM01, U3 CC2541

Commit message: PCB layout done
Parts:
- removed JP2: (no value), pinhead:2X05
- removed R3: 10k, rcl:R0603
- removed S1: (no value), switch-tact:DTSM-3
- added J1: ICSP, SHF-105-01-X-D-SM:SHF-105-01-X-D-SM
- added R1: (no value), smd-ipc:C0402
- added S2: (no value), Push Button:434121050816
- C1, C26, C28, C29, C30, C31, C7: value 100nF -> (none)
- C18, C19: value 18pF -> (none)
- C2, C5: value 10uF -> (none)
- C21, C22, C24: value 1pF -> (none)
- C23: value DNM -> (none)
- C25: value 220pF -> (none)
- C27, C32: value 1uF -> (none)
- C33, C34: value 12pF -> (none)
- C35, C36: value 15pF -> (none)
- C6: value 2.2uF -> (none)
- C9: value 100n -> (none)
- L1, L2: value 2nH -> (none)
- L3: value 1nH -> (none)
- L4: value 3nH -> (none)
- L5: value BLM15HG102SN1D -> (none)
- Q3: value 32-MHz -> (none)
- Q4: value 32.768-kHz -> (none)
- R10: value 56k -> (none)
- R2, R7: value 10k -> (none)
- R4: value 1k -> (none); device rcl:R0603 -> smd-ipc:C0402
- R8: value 2.7k -> (none)
- T1: value BC848 -> (none)
- U1: value LM1117-3.3 -> (none)
- U3: value CC2541 -> (none)
- moved C6 64.3 mm to (6.19, 12.3), turned to 180 degrees
- moved L5 62.9 mm to (10.0, 12.3), turned to 180 degrees
- moved C2 52.5 mm to (2.76, 13.8), turned to 0 degrees
- moved C1 49.8 mm to (2.76, 16.2), turned to 0 degrees
- moved R7 46.6 mm to (17.7, 21.4), turned to 180 degrees
- moved C5 46.2 mm to (2.76, 18.5), turned to 0 degrees
- moved U1 45.2 mm to (8.90, 16.2), turned to 90 degrees
- moved R2 45.2 mm to (23.0, 22.2)
- moved C7 43.2 mm to (2.76, 20.6), turned to 0 degrees
- moved R4 39.6 mm to (16.7, 18.2), turned to 180 degrees
- moved T1 31.7 mm to (14.6, 23.8), turned to 0 degrees
- moved X1 27.0 mm to (4.30, 31.8), turned to 90 degrees
- moved LED1 17.5 mm to (14.3, 4.99), flipped to the top, turned to 270 degrees
- moved K1 9.61 mm to (22.4, 33.8)
- moved F2 8.72 mm to (30.2, 40.7), turned to 90 degrees
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Connections:
- removed net +4.1V: C25.1, C26.1, C28.1, C29.1, C30.1, C31.1, C32.1, C6.1, JP2.2, L5.1, R2.2, R7.2, SJ1.2, U3.10, U3.21, U3.24, U3.27, U3.28, U3.29, U3.31, U3.39
- new net 3.3: C1.1, C2.1, L5.2, U1.2, U1.4
- net 3.3V: now also C25.1, C26.1, C28.1, C29.1, C30.1, C31.1, C32.1, C6.1, J1.2, L5.1, R2.2, R7.2, SJ1.2, U3.10, U3.21, U3.24, U3.27, U3.28, U3.29, U3.31, U3.39; no longer C1.1, C2.1, L5.2, U1.2, U1.4
- net BUTTON_PROG: now also S2.2; no longer S1.2
- net DEBUG_CLK: now also J1.3; no longer JP2.3
- net DEBUG_DATA: now also J1.4; no longer JP2.4
- net DEBUG_RESET: now also J1.7; no longer JP2.7
- net GND: now also J1.1, S2.1; no longer JP2.1, S1.1
- net LED_STATUS: now also R4.2, U3.36; no longer R3.1, U3.11
- net LOAD_CONTROL: now also R1.2; no longer R4.1
- net N$1: now also R4.1; no longer R3.2
- net N$10: now also J1.9; no longer JP2.9
- net N$6: now also R1.1; no longer R4.2
Routing:
- net 3.3V: track 0.00 -> 100.4 mm, vias 0 -> 8
- net N$3: track 0.00 -> 46.5 mm
- net L1_PHASE: track 0.00 -> 42.6 mm
- net N$4: track 0.00 -> 38.4 mm
- net DEBUG_RESET: track 0.00 -> 34.3 mm, vias 0 -> 3
- net PHY_SWITCH_STATUS: track 0.00 -> 33.0 mm
- net 5V: track 0.00 -> 30.1 mm
- net BUTTON_PROG: track 0.00 -> 27.3 mm, vias 0 -> 3
- net N$9: track 0.00 -> 24.2 mm
- net GND: track 0.00 -> 19.7 mm, vias 0 -> 121
- net N$8: track 0.00 -> 18.2 mm
- net N$1: track 0.00 -> 15.0 mm, vias 0 -> 3
- net 3.3: track 0.00 -> 14.8 mm
- net +4.1V: track 13.6 -> 0.00 mm
- net N$6: track 0.00 -> 9.49 mm
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- added copper zone on layer 1, net GND
- added copper zone on layer 16, net GND
Other:
- board text added: "WorkshySwitch"
- board text added: "open source hardware"
